File: hc_real_pad.kicad_pcb (KiCad board)
At the start: 2 copper layers, 74.4 x 45.2 mm, 55 parts, among them J1 OLED_DISPLAY, SW1 SW_Push_45deg, SW10 SW_Push_45deg, SW11 SW_Push_45deg, SW12 SW_Push_45deg, SW13 SW_Push_45deg, SW14 SW_Push_45deg, SW15 SW_Push_45deg, SW16 SW_Push_45deg, SW17 RotaryEncoder_Switch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

Commit message: finished making the pcb
Parts:
- D1, D10, D11, D12, D13, D14, D15, D16, D17, D18, D2, D3, D4, D5, D6, D7, D8, D9: moved to B.Cu
- moved D17 179.0 mm to (201.9, 115.6), turned to -90 degrees
- moved D18 177.5 mm to (201.9, 111.8), turned to 90 degrees
- moved D16 175.2 mm to (174.0, 168.9), turned to 180 degrees
- moved D12 168.4 mm to (154.9, 168.9), turned to 180 degrees
- moved D15 167.2 mm to (174.0, 149.9), turned to 180 degrees
- moved D8 164.9 mm to (135.9, 168.9), turned to 180 degrees
- moved D4 164.7 mm to (116.8, 168.9), turned to 180 degrees
- moved D14 160.4 mm to (174.0, 130.8), turned to 180 degrees
- moved D11 158.8 mm to (154.9, 149.9), turned to 180 degrees
- moved D13 154.8 mm to (174.0, 111.8), turned to 180 degrees
- moved D7 153.5 mm to (135.9, 149.9), turned to 180 degrees
- moved D3 151.9 mm to (116.8, 149.9), turned to 180 degrees
- moved D10 150.1 mm to (154.9, 130.8), turned to 180 degrees
- moved D6 143.0 mm to (135.9, 130.8), turned to 180 degrees
- moved D9 142.6 mm to (154.9, 111.8), turned to 180 degrees
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Connections:
- J1 pad 1: SDA -> GND
- J1 pad 2: SCL -> VCC
- J1 pad 3: VCC -> SCL
- J1 pad 4: GND -> SDA
Routing:
- net ENCSWB0: track 0.00 -> 240.6 mm
- net ENCSWA0: track 0.00 -> 240.0 mm
- net GND: track 123.0 -> 345.3 mm
- net ROW3: track 0.00 -> 185.9 mm
- net ROW0: track 0.00 -> 181.3 mm
- net COL4: track 0.00 -> 135.5 mm, vias 0 -> 2
- net ENCSWA1: track 0.00 -> 133.9 mm, vias 0 -> 1
- net ENCSWB1: track 0.00 -> 132.7 mm, vias 0 -> 1
- net ROW2: track 0.00 -> 130.5 mm
- net ROW1: track 0.00 -> 110.4 mm
- net SDA: track 0.00 -> 106.6 mm
- net SCL: track 0.00 -> 98.9 mm
- net COL3: track 0.00 -> 97.8 mm
- net COL0: track 0.00 -> 97.5 mm
- net COL1: track 0.00 -> 87.9 mm
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Other:
- board size 74.4 x 45.2 mm -> 149.9 x 81.3 mm
- board text added: "Daniel Pitman"
- board text added: "Feb 26"
- board text added: "LET THERE BE LIGHT"
- board text added: "MEGAPAD"
- board text added: "SHOW ME WHAT I NEED TO KNOW"
- board text added: "UNLOCK YOUR SPEED"
